File: circuit/analog.sch (EAGLE design)
At the start: 44 parts, among them IC1 AD8532, IC2 74HC4052D, IC3 AD8532, IC4 4066D, IC5 4066D

Commit message: - будем полностью перерисовывать под другие усилители , AD8532 имеет слишком высокий Input offset voltage.
Parts:
- added C14: 100n, rcl:C-EUC0603
Connections:
- net GNDA: now also C14.1
- net N$9: now also C14.2
Changed lines of the file:
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@@
 <part name="GND13" library="supply1" deviceset="GNDA" device=""/>
 <part name="GND14" library="supply1" deviceset="GNDA" device=""/>
+<part name="C14" library="rcl" deviceset="C-EU" device="C0603" value="100n"/>
 </parts>
 <sheets>
@@
 <instance part="GND13" gate="1" x="152.4" y="-73.66"/>
 <instance part="GND14" gate="1" x="-33.02" y="-33.02"/>
+<instance part="C14" gate="G$1" x="27.94" y="30.48" rot="R180"/>
 </instances>
 <busses>
@@
 <pinref part="R7" gate="G$1" pin="1"/>
 <pinref part="GND6" gate="1" pin="GNDA"/>
+<pinref part="C14" gate="G$1" pin="1"/>
+<wire x1="33.02" y1="25.4" x2="27.94" y2="25.4" width="0.1524" layer="91"/>
+<wire x1="27.94" y1="25.4" x2="27.94" y2="27.94" width="0.1524" layer="91"/>
+<junction x="33.02" y="25.4"/>
 </segment>
 <segment>
@@
 <pinref part="R7" gate="G$1" pin="2"/>
 <junction x="33.02" y="35.56"/>
-</segment>
-</net>
+<pinref part="C14" gate="G$1" pin="2"/>
+<wire x1="33.02" y1="35.56" x2="27.94" y2="35.56" width="0.1524" layer="91"/>
+</segment>
+</net>
