File: circuit/analog3.sch (EAGLE design)
At the start: 73 parts, among them IC1 AD8603UJ, IC2 74HC4052D, IC3 AD8603UJ, IC4 AD8221R, IC5 AD8221R, IC6 LM258, IC7 LM258

Commit message: - на цифровой схеме добавили разъем для Nokia 5110, коннекторы для переключения питания, объединили восточный разъем - на аналоговой схеме добавили включение 3.3 nF конденсатор, для фильтрации высокочастотных шумов ADC
Parts:
- added C7: 3.3n, rcl:C-EUC0805
- added U$1: SN74LVC1G3157DBVR, balmer:SN74LVC1G3157DBVR
- C2: value 33p -> 68p
Connections:
- new net ANALOG_SW: U$1.S, X8-2.1
- new net N$7: C7.1, U$1.B1
- net +5V: now also U$1.VCC
- net GNDA: now also C7.2, U$1.GND
- net N$3: now also U$1.A
Changed lines of the file:
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@@
 <layer number="48" name="Document" color="7" fill="1" visible="no" active="no"/>
 <layer number="49" name="Reference" color="7" fill="1" visible="no" active="no"/>
+<layer number="50" name="dxf" color="7" fill="1" visible="no" active="no"/>
 <layer number="51" name="tDocu" color="7" fill="1" visible="no" active="no"/>
 <layer number="52" name="bDocu" color="7" fill="1" visible="no" active="no"/>
+<layer number="53" name="tGND_GNDA" color="7" fill="9" visible="no" active="no"/>
+<layer number="54" name="bGND_GNDA" color="1" fill="9" visible="no" active="no"/>
+<layer number="56" name="wert" color="7" fill="1" visible="no" active="no"/>
 <layer number="91" name="Nets" color="2" fill="1" visible="yes" active="yes"/>
 <layer number="92" name="Busses" color="1" fill="1" visible="yes" active="yes"/>
@@
 <layer number="97" name="Info" color="7" fill="1" visible="yes" active="yes"/>
 <layer number="98" name="Guide" color="6" fill="1" visible="yes" active="yes"/>
+<layer number="100" name="Muster" color="7" fill="1" visible="no" active="no"/>
+<layer number="101" name="Patch_Top" color="12" fill="4" visible="yes" active="yes"/>
+<layer number="102" name="Vscore" color="7" fill="1" visible="yes" active="yes"/>
+<layer number="103" name="tMap" color="7" fill="1" visible="yes" active="yes"/>
+<layer number="104" name="Name" color="16" fill="1" visible="yes" active="yes"/>
+<layer number="105" name="tPlate" color="7" fill="1" visible="yes" active="yes"/>
+<layer number="106" name="bPlate" color="7" fill="1" visible="yes" active="yes"/>
+<layer number="107" name="Crop" color="7" fill="1" visible="yes" active="yes"/>
+<layer number="108" name="tplace-old" color="10" fill="1" visible="yes" active="yes"/>
+<layer number="109" name="ref-old" color="11" fill="1" visible="yes" active="yes"/>
+<layer number="116" name="Patch_BOT" color="9" fill="4" visible="yes" active="yes"/>
+<layer number="121" name="_tsilk" color="7" fill="1" visible="yes" active="yes"/>
+<layer number="122" name="_bsilk" color="7" fill="1" visible="yes" active="yes"/>
+<layer number="125" name="_tNames" color="7" fill="1" visible="yes" active="yes"/>
+<layer number="144" name="Drill_legend" color="7" fill="1" visible="yes" active="yes"/>
+<layer number="151" name="HeatSink" color="7" fill="1" visible="yes" active="yes"/>
+<layer number="199" name="Contour" color="7" fill="1" visible="yes" active="yes"/>
+<layer number="200" name="200bmp" color="1" fill="10" visible="yes" active="yes"/>
+<layer number="201" name="201bmp" color="2" fill="10" visible="yes" active="yes"/>
+<layer number="202" name="202bmp" color="3" fill="10" visible="yes" active="yes"/>
+<layer number="203" name="203bmp" color="4" fill="10" visible="yes" active="yes"/>
+<layer number="204" name="204bmp" color="5" fill="10" visible="yes" active="yes"/>
+<layer number="205" name="205bmp" color="6" fill="10" visible="yes" active="yes"/>
+<layer number="206" name="206bmp" color="7" fill="10" visible="yes" active="yes"/>
+<layer number="207" name="207bmp" color="8" fill="10" visible="yes" active="yes"/>
+<layer number="208" name="208bmp" color="9" fill="10" visible="yes" active="yes"/>
+<layer number="209" name="209bmp" color="7" fill="1" visible="yes" active="yes"/>
+<layer number="210" name="210bmp" color="7" fill="1" visible="yes" active="yes"/>
+<layer number="211" name="211bmp" color="7" fill="1" visible="yes" active="yes"/>
+<layer number="212" name="212bmp" color="7" fill="1" visible="yes" active="yes"/>
+<layer number="213" name="213bmp" color="7" fill="1" visible="yes" active="yes"/>
+<layer number="214" name="214bmp" color="7" fill="1" visible="yes" active="yes"/>
+<layer number="215" name="215bmp" color="7" fill="1" visible="yes" active="yes"/>
+<layer number="216" name="216bmp" color="7" fill="1" visible="yes" active="yes"/>
+<layer number="217" name="217bmp" color="18" fill="1" visible="no" active="no"/>
+<layer number="218" name="218bmp" color="19" fill="1" visible="no" active="no"/>
+<layer number="219" name="219bmp" color="20" fill="1" visible="no" active="no"/>
+<layer number="220" name="220bmp" color="21" fill="1" visible="no" active="no"/>
+<layer number="221" name="221bmp" color="22" fill="1" visible="no" active="no"/>
+<layer number="222" name="222bmp" color="23" fill="1" visible="no" active="no"/>
+<layer number="223" name="223bmp" color="24" fill="1" visible="no" active="no"/>
+<layer number="224" name="224bmp" color="25" fill="1" visible="no" active="no"/>
+<layer number="250" name="Descript" color="3" fill="1" visible="no" active="no"/>
+<layer number="251" name="SMDround" color="12" fill="11" visible="no" active="no"/>
+<layer number="254" name="cooling" color="7" fill="1" visible="yes" active="yes"/>
 </layers>
 <schematic xreflabel="%F%N/%S.%C%R" xrefpart="/%S.%C%R">
@@
 <parts>
 <part name="R2" library="rcl" deviceset="R-EU_" device="R0603" value="12k"/>
-<part name="C2" library="rcl" deviceset="C-EU" device="C0805" value="33p"/>
+<part name="C2" library="rcl" deviceset="C-EU" device="C0805" value="68p"/>
 <part name="C4" library="rcl" deviceset="C-EU" device="C0603" value="1mk"/>
 <part name="C5" library="rcl" deviceset="C-EU" device="C0603" value="100n"/>
@@
 <part name="P+9" library="supply1" deviceset="+5V" device=""/>
 <part name="C1" library="rcl" deviceset="C-EU" device="C0805" value="10mk"/>
+<part name="U$1" library="balmer" deviceset="SN74LVC1G3157DBVR" device=""/>
+<part name="GND24" library="supply1" deviceset="GNDA" device=""/>
+<part name="P+10" library="supply1" deviceset="+5V" device=""/>
+<part name="C7" library="rcl" deviceset="C-EU" device="C0805" value="3.3n"/>
+<part name="GND25" library="supply1" deviceset="GNDA" device=""/>
 </parts>
 <sheets>
@@
 <instance part="P+9" gate="1" x="86.36" y="76.2"/>
 <instance part="C1" gate="G$1" x="63.5" y="-101.6"/>
+<instance part="U$1" gate="G$1" x="0" y="99.06"/>
+<instance part="GND24" gate="1" x="-2.54" y="86.36"/>
+<instance part="P+10" gate="1" x="-2.54" y="111.76"/>
+<instance part="C7" gate="G$1" x="12.7" y="104.14" rot="R90"/>
+<instance part="GND25" gate="1" x="22.86" y="101.6"/>
 </instances>
 <busses>
@@
 <wire x1="-22.86" y1="78.74" x2="-35.56" y2="78.74" width="0.1524" layer="91"/>
 <junction x="-22.86" y="78.74"/>
+<wire x1="-22.86" y1="78.74" x2="-22.86" y2="99.06" width="0.1524" layer="91"/>
+<pinref part="U$1" gate="G$1" pin="A"/>
+<wire x1="-22.86" y1="99.06" x2="-10.16" y2="99.06" width="0.1524" layer="91"/>
 </segment>
 </net>
@@
 <pinref part="IC6" gate="P" pin="V+"/>
 <pinref part="P+9" gate="1" pin="+5V"/>
+</segment>
+<segment>
+<pinref part="U$1" gate="G$1" pin="VCC"/>
+<pinref part="P+10" gate="1" pin="+5V"/>
 </segment>
 </net>
@@
 <pinref part="IC1" gate="G$1" pin="-VS"/>
 <wire x1="-43.18" y1="68.58" x2="-43.18" y2="71.12" width="0.1524" layer="91"/>
+</segment>
+<segment>
+<pinref part="U$1" gate="G$1" pin="GND"/>
+<pinref part="GND24" gate="1" pin="GNDA"/>
+</segment>
+<segment>
+<pinref part="C7" gate="G$1" pin="2"/>
+<pinref part="GND25" gate="1" pin="GNDA"/>
+<wire x1="17.78" y1="104.14" x2="22.86" y2="104.14" width="0.1524" layer="91"/>
 </segment>
 </net>
@@
 </segment>
 </net>
+<net name="ANALOG_SW" class="0">
+<segment>
+<pinref part="X8" gate="-2" pin="1"/>
+<wire x1="149.86" y1="88.9" x2="139.7" y2="88.9" width="0.1524" layer="91"/>
+<label x="134.366" y="89.408" size="1.778" layer="95"/>
+</segment>
+<segment>
+<pinref part="U$1" gate="G$1" pin="S"/>
+<wire x1="10.16" y1="93.98" x2="22.86" y2="93.98" width="0.1524" layer="91"/>
+<label x="11.43" y="94.742" size="1.778" layer="95"/>
+</segment>
+</net>
+<net name="N$7" class="0">
+<segment>
+<pinref part="U$1" gate="G$1" pin="B1"/>
+<pinref part="C7" gate="G$1" pin="1"/>
+</segment>
+</net>
